Commit message: attached grippers to digit's arms

File: morpheus/models/fetch_description/robots/freight.urdf (robot description, URDF)
Before this commit: robot freight, 7 links, 6 joints
Links:
- added link lift, mass 7.1294; collision box size=0.2 0.2 0.4; visual box size=0.2 0.2 0.4
- added link pedestal, mass 7.1294; collision box size=0.3 0.3 1.0; visual box size=0.25 0.25 0.6
Joints:
- added joint base_to_pedestal: type fixed, parent base_link, child pedestal, origin xyz=0 0 0.6 rpy=0 0 0
- added joint pedestal_to_lift: type prismatic, parent pedestal, child lift, origin xyz=0 0 0.2 rpy=0 0 0, axis 0 0 1, limit lower=0.0 upper=0.3 effort=30000 velocity=1000

File: morpheus/models/yumi_description/yumi_grippers.urdf (robot description, URDF)
Before this commit: robot yumi, 23 links, 22 joints
Links:
- removed link table_top
- link yumi_body: mass 15 -> 5
Joints:
- removed joint yumi_body_to_table_top
