Commit message: implemented top grasp and side grasp

File: digit/models/buff_digit/digit_husky.urdf (robot description, URDF)
Before this commit: robot buff_digit, 43 links, 42 joints
Links:
- removed link base_camera_link
- removed link base_camera_optical_frame
- removed link estop_link
- removed link l_wheel_link
- removed link laser_link
- removed link r_wheel_link
- added link front_bumper_link; visual box size=0.001 0.001 0.001
- added link front_left_wheel_link, mass 2.637; collision cylinder length=0.1143 radius=0.17775; visual box size=0.001 0.001 0.001
- added link front_right_wheel_link, mass 2.637; collision cylinder length=0.1143 radius=0.17775; visual box size=0.001 0.001 0.001
- added link imu_link
- added link rear_bumper_link; visual box size=0.001 0.001 0.001
- added link rear_left_wheel_link, mass 2.637; collision cylinder length=0.1143 radius=0.17775; visual box size=0.001 0.001 0.001
- added link rear_right_wheel_link, mass 2.637; collision cylinder length=0.1143 radius=0.17775; visual box size=0.001 0.001 0.001
- added link top_plate_link; visual box size=0.001 0.001 0.001
- added link user_rail_link; visual box size=0.001 0.001 0.001
- link base_link: mass 100.1294 -> 33.455; geometry collision box size=1.0074 0.5709 0.2675; visual box size=0.001 0.001 0.001
Joints:
- removed joint base_camera_joint
- removed joint base_camera_optical_joint
- removed joint estop_joint
- removed joint l_wheel_joint
- removed joint laser_joint
- removed joint r_wheel_joint
- added joint front_bumper: type fixed, parent base_link, child front_bumper_link, origin xyz=0.48 0 0.091 rpy=0 0 0
- added joint front_left_wheel: type continuous, parent base_link, child front_left_wheel_link, origin xyz=0.256 0.2854 0.03282 rpy=0 0 0, axis 0 1 0
- added joint front_right_wheel: type continuous, parent base_link, child front_right_wheel_link, origin xyz=0.256 -0.2854 0.03282 rpy=0 0 0, axis 0 1 0
- added joint imu_joint: type fixed, parent base_link, child imu_link, origin xyz=$(optenv HUSKY_IMU_XYZ 0.19 0 0.149) rpy=$(optenv HUSKY_IMU_RPY 0 -1.5708 3.1416)
- added joint rear_bumper: type fixed, parent base_link, child rear_bumper_link, origin xyz=-0.48 0 0.091 rpy=0 0 3.14159
- added joint rear_left_wheel: type continuous, parent base_link, child rear_left_wheel_link, origin xyz=-0.256 0.2854 0.03282 rpy=0 0 0, axis 0 1 0
- added joint rear_right_wheel: type continuous, parent base_link, child rear_right_wheel_link, origin xyz=-0.256 -0.2854 0.03282 rpy=0 0 0, axis 0 1 0
- added joint top_plate: type fixed, parent base_link, child top_plate_link
- added joint user_rail: type fixed, parent base_link, child user_rail_link, origin xyz=0.272 0 0.245 rpy=0 0 0
- joint digit_to_freight: origin xyz=0 0  0.9 rpy=0 0 0 -> xyz=0 0  0.7 rpy=0 0 0

File: digit/models/table/table.urdf (robot description, URDF)
Before this commit: robot table.urdf, 1 links, 0 joints
Links:
- link baseLink: geometry collision box size=1.5 1 0.05; visual mesh filename=table.obj scale=0.1 0.1 0.9
