Commit message: ikfast working with dual digit arms

File: digit/models/buff_digit/left_prosthetic.urdf (robot description, URDF)
Before this commit: robot prosthetic, 12 links, 11 joints
Links:
- removed link right_gripper_base
- removed link right_gripper_ee
- removed link right_jlink0
- removed link right_jlink1
- removed link right_jlink2
- removed link right_jlink3
- removed link right_jlink4
- removed link right_link1
- removed link right_link2
- removed link right_link3
- removed link right_link4
- removed link right_wrist
- added link left_gripper_base, mass 0.2; collision cylinder length=0.1 radius=0.04; visual cylinder length=0.1 radius=0.04
- added link left_gripper_ee, mass 0.2; collision cylinder length=0.025 radius=0.025; visual cylinder length=0.025 radius=0.025
- added link left_jlink0, mass .01; collision cylinder length=0.025 radius=0.025; visual cylinder length=0.025 radius=0.025
- added link left_jlink1, mass .01; collision cylinder length=0.025 radius=0.025; visual cylinder length=0.025 radius=0.025
- added link left_jlink2, mass .01; collision cylinder length=0.025 radius=0.025; visual cylinder length=0.025 radius=0.025
- added link left_jlink3, mass .01; collision cylinder length=0.025 radius=0.025; visual cylinder length=0.025 radius=0.025
- added link left_jlink4, mass 0.550582; collision cylinder length=0.025 radius=0.025; visual cylinder length=0.025 radius=0.025
- added link left_link1, mass .000000001; collision cylinder length=0.08 radius=0.0125; visual cylinder length=0.08 radius=0.0125
- added link left_link2, mass .000000001; collision cylinder length=0.2 radius=0.03; visual cylinder length=0.2 radius=0.03
- added link left_link3, mass .000000001; collision cylinder length=0.2 radius=0.03; visual cylinder length=0.2 radius=0.03
- added link left_link4, mass .000000001; collision cylinder length=0.4 radius=0.03; visual cylinder length=0.4 radius=0.03
- added link left_wrist, mass 0.550582; collision cylinder length=0.05 radius=0.025; visual cylinder length=0.05 radius=0.025
Joints:
- removed joint gripper_right_wrist_joint
- removed joint right_gripper_baseee_to_gripper_base
- removed joint right_joint1
- removed joint right_joint1f
- removed joint right_joint2
- removed joint right_joint2f
- removed joint right_joint3
- removed joint right_joint3f
- removed joint right_joint4
- removed joint right_joint4f
- removed joint right_wrist_joint
- added joint gripper_left_wrist_joint: type revolute, parent left_wrist, child left_gripper_base, origin xyz=0.07 0 0 rpy=0 0 0, axis 1 0 0, limit lower=-1.57 upper=1.57 effort=1.4 velocity=10
- added joint left_gripper_baseee_to_gripper_base: type fixed, parent left_gripper_base, child left_gripper_ee, origin xyz=0.05125 0.0 0 rpy=0 0 0
- added joint left_joint1: type revolute, parent left_link1, child left_jlink1, origin xyz=0 0.04 0 rpy=0 0 0, axis 1 0 0, limit lower=-3.1415 upper=3.1415 effort=1.4 velocity=0.25
- added joint left_joint1f: type revolute, parent left_jlink0, child left_link1, origin xyz=0 0.04 0.0 rpy=0 0 0, axis 0 1 0, limit lower=-3.1415 upper=3.1415 effort=1.4 velocity=0.25
- added joint left_joint2: type fixed, parent left_link2, child left_jlink2, origin xyz=0 0 -0.1 rpy=0 0 0
- added joint left_joint2f: type fixed, parent left_jlink1, child left_link2, origin xyz=0 0  -0.1 rpy=0 0 0
- added joint left_joint3: type revolute, parent left_link3, child left_jlink3, origin xyz=0 0.0 -0.1 rpy=0 0 0, axis 1 0 0, limit lower=-3.1415 upper=3.1415 effort=1.4 velocity=0.25
- added joint left_joint3f: type fixed, parent left_jlink2, child left_link3, origin xyz=0 0  -0.1035 rpy=0 0 0
- added joint left_joint4: type revolute, parent left_link4, child left_jlink4, origin xyz=0.0 0.0 -0.2 rpy=0 0 0, axis 0 0 1, limit lower=-1.57 upper=1.57 effort=1.4 velocity=10
- added joint left_joint4f: type fixed, parent left_jlink3, child left_link4, origin xyz=0 0  -0.2 rpy=0 0 0
- added joint left_wrist_joint: type revolute, parent left_jlink4, child left_wrist, origin xyz=0.0 0.0 -0.025 rpy=0 1.5707 0, axis 0 1 0, limit lower=-1.57 upper=1.57 effort=1.4 velocity=10

File: digit/models/buff_digit/prost_digit_freight.urdf (robot description, URDF)
Before this commit: robot buff_digit, 43 links, 42 joints
Links:
- removed link gripper_r_base
- removed link right_elbow
- removed link right_shoulder_pitch
- removed link right_shoulder_roll
- removed link right_shoulder_yaw
- added link left_attach, mass .01; collision cylinder length=0.1 radius=0.025; visual cylinder length=0.1 radius=0.025
- added link left_jlink4, mass 0.550582; collision cylinder length=0.025 radius=0.025; visual cylinder length=0.025 radius=0.025
- added link right_attach, mass .01; collision cylinder length=0.1 radius=0.025; visual cylinder length=0.1 radius=0.025
- added link right_gripper_base, mass 0.2; collision cylinder length=0.1 radius=0.04; visual cylinder length=0.1 radius=0.04
- added link right_jlink0, mass .01; collision cylinder length=0.025 radius=0.025; visual cylinder length=0.025 radius=0.025
- added link right_jlink1, mass .01; collision cylinder length=0.025 radius=0.025; visual cylinder length=0.025 radius=0.025
- added link right_jlink2, mass .01; collision cylinder length=0.025 radius=0.025; visual cylinder length=0.025 radius=0.025
- added link right_jlink3, mass .01; collision cylinder length=0.025 radius=0.025; visual cylinder length=0.025 radius=0.025
- added link right_jlink4, mass 0.550582; collision cylinder length=0.025 radius=0.025; visual cylinder length=0.025 radius=0.025
- added link right_link1, mass .000000001; collision cylinder length=0.08 radius=0.0125; visual cylinder length=0.08 radius=0.0125
- added link right_link2, mass .000000001; collision cylinder length=0.2 radius=0.03; visual cylinder length=0.2 radius=0.03
- added link right_link3, mass .000000001; collision cylinder length=0.2 radius=0.03; visual cylinder length=0.2 radius=0.03
- added link right_link4, mass .000000001; collision cylinder length=0.4 radius=0.03; visual cylinder length=0.4 radius=0.03
- link left_jlink0: mass 0.535396 -> .01; geometry collision cylinder length=0.025 radius=0.025; visual cylinder length=0.025 radius=0.025
- link left_jlink1: mass 1.065387 -> .01
- link left_link1: mass 1.440357 -> .000000001; geometry collision cylinder length=0.08 radius=0.0125; visual cylinder length=0.08 radius=0.0125
- link left_link2: mass 0.550582 -> .000000001
- link left_link3: mass 0.550582 -> .000000001
- link left_link4: mass 0.550582 -> .000000001
- link right_gripper_ee: mass None -> 0.2; geometry collision cylinder length=0.025 radius=0.025; visual cylinder length=0.025 radius=0.025
Joints:
- removed joint elbow_joint_right
- removed joint left_gripper_ee_to_gripper_base
- removed joint right_ee_to_gripper_base
- removed joint shoulder_pitch_joint_right
- removed joint shoulder_roll_joint_left
- removed joint shoulder_roll_joint_right
- removed joint shoulder_yaw_joint_right
- added joint left_arm_to_left_attach: type fixed, parent left_attach, child left_jlink0, origin xyz=0 0 0 rpy=0 0 0
- added joint left_attach_to_torso: type fixed, parent torso, child left_attach, origin xyz=-0.001 0.12 0.4 rpy=0 0 0
- added joint left_gripper_baseee_to_gripper_base: type fixed, parent left_gripper_base, child left_gripper_ee, origin xyz=0.05125 0.0 0 rpy=0 0 0
- added joint left_joint4: type revolute, parent left_link4, child left_jlink4, origin xyz=0.0 0.0 -0.2 rpy=0 0 0, axis 0 0 1, limit lower=-1.57 upper=1.57 effort=1.4 velocity=10
- added joint right_arm_to_right_attach: type fixed, parent right_attach, child right_jlink0, origin xyz=0 0 0 rpy=0 0 0
- added joint right_attach_to_torso: type fixed, parent torso, child right_attach, origin xyz=-0.001 -0.12 0.4 rpy=0 0 0
- added joint right_gripper_baseee_to_gripper_base: type fixed, parent right_gripper_base, child right_gripper_ee, origin xyz=0.05125 0.0 0 rpy=0 0 0
- added joint right_joint1: type revolute, parent right_link1, child right_jlink1, origin xyz=0 -0.04 0 rpy=0 0 0, axis 1 0 0, limit lower=-3.1415 upper=3.1415 effort=1.4 velocity=0.25
- added joint right_joint1f: type revolute, parent right_jlink0, child right_link1, origin xyz=0 -0.04 0.0 rpy=0 0 0, axis 0 1 0, limit lower=-3.1415 upper=3.1415 effort=1.4 velocity=0.25
- added joint right_joint2: type fixed, parent right_link2, child right_jlink2, origin xyz=0 0 -0.1 rpy=0 0 0
- added joint right_joint2f: type fixed, parent right_jlink1, child right_link2, origin xyz=0 0  -0.1 rpy=0 0 0
- added joint right_joint3: type revolute, parent right_link3, child right_jlink3, origin xyz=0 0.0 -0.1 rpy=0 0 0, axis 1 0 0, limit lower=-3.1415 upper=3.1415 effort=1.4 velocity=0.25
- added joint right_joint3f: type fixed, parent right_jlink2, child right_link3, origin xyz=0 0  -0.1035 rpy=0 0 0
- added joint right_joint4: type revolute, parent right_link4, child right_jlink4, origin xyz=0.0 0.0 -0.2 rpy=0 0 0, axis 0 0 1, limit lower=-1.57 upper=1.57 effort=1.4 velocity=10
- added joint right_joint4f: type fixed, parent right_jlink3, child right_link4, origin xyz=0 0  -0.2 rpy=0 0 0
- joint gripper_right_wrist_joint: child gripper_r_base -> right_gripper_base; limit lower=-1.57 upper=1.57 effort=0 velocity=10 -> lower=-1.57 upper=1.57 effort=1.4 velocity=10; origin xyz=0.02 0 0 rpy=0 0 0 -> xyz=0.07 0 0 rpy=0 0 0
- joint left_joint1: axis 0 1 0 -> 1 0 0; limit lower=-1.7453 upper=1.7453 effort=1.4 velocity=10 -> lower=-3.1415 upper=3.1415 effort=1.4 velocity=0.25; origin xyz=0 0.04 0 rpy=0 0.785398163397 0 -> xyz=0 0.04 0 rpy=0 0 0; type continuous -> revolute
- joint left_joint1f: axis (none) -> 0 1 0; limit (none) -> lower=-3.1415 upper=3.1415 effort=1.4 velocity=0.25; origin xyz=0 0.04 0.00625 rpy=0 0 0 -> xyz=0 0.04 0.0 rpy=0 0 0; type fixed -> revolute
- joint left_joint2: axis 0 0 1 -> (none); limit lower=-1.3526 upper=1.3526 effort=1.4 velocity=12.5 -> (none); type continuous -> fixed
- joint left_joint3: axis 0 1 0 -> 1 0 0; origin xyz=0 0.025 -0.1 rpy=0 -1.06 0 -> xyz=0 0.0 -0.1 rpy=0 0 0; type continuous -> revolute
- joint left_wrist_joint: origin xyz=0.0 0.0 -0.22 rpy=0 1.5707 0 -> xyz=0.0 0.0 -0.025 rpy=0 1.5707 0; parent left_link4 -> left_jlink4
- joint right_wrist_joint: limit lower=-1.57 upper=1.57 effort=0 velocity=10 -> lower=-1.57 upper=1.57 effort=1.4 velocity=10; origin xyz=0.38 -0.0 -0.06 rpy=-1.57079632679 0.1926991 0 -> xyz=0.0 0.0 -0.025 rpy=0 1.5707 0; parent right_elbow -> right_jlink4
