Commit message: camera working

File: digit/models/buff_digit/prost_digit_hover.urdf (robot description, URDF)
Before this commit: robot buff_digit, 52 links, 51 joints
Links:
- removed link base_camera_link
- removed link base_camera_optical_frame
- removed link estop_link
- removed link footprint
- removed link l_wheel_link
- removed link laser_link
- removed link r_wheel_link
- added link left_wheel, mass 4.028392; collision box size=0.005 0.005 0.005; visual mesh filename=/home/bill/garage/kfp_v2/digit/models/hoverboard/meshes/whe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 scale=0.025 0.025 0.025
- added link right_wheel, mass 4.028392; collision box size=0.005 0.005 0.005; visual mesh filename=/home/bill/garage/kfp_v2/digit/models/hoverboard/meshes/whe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 scale=0.025 0.025 0.025
- link base_link: mass 100.1294 -> 15.028392; geometry collision box size=0.5 0.15 0.5; visual mesh filename=/home/bill/garage/kfp_v2/digit/models/hoverboard/meshes/bas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 scale=0.025 0.025 0.025
Joints:
- removed joint base_camera_joint
- removed joint base_camera_optical_joint
- removed joint estop_joint
- removed joint footprint_to_base
- removed joint l_wheel_joint
- removed joint laser_joint
- removed joint r_wheel_joint
- added joint wheell_to_base: type fixed, parent base_link, child left_wheel, origin xyz=0 1.0 0 rpy=0 0 0, axis 0 1 0, limit effort=8.85 velocity=34.8
- added joint wheelr_to_base: type continuous, parent base_link, child right_wheel, origin xyz=0 0 0 rpy=0 0 3.14159265359, axis 0 1 0, limit effort=8.85 velocity=34.8
- joint hip_abduction_left: type continuous -> fixed
- joint hip_abduction_right: type continuous -> fixed
- joint hip_flexion_left: type continuous -> fixed
- joint hip_flexion_right: type continuous -> fixed
- joint hip_rotation_left: type continuous -> fixed
- joint hip_rotation_right: type continuous -> fixed
- joint knee_joint_left: type continuous -> fixed
- joint knee_joint_right: type continuous -> fixed
- joint knee_to_shin_left: type continuous -> fixed
- joint knee_to_shin_right: type continuous -> fixed
- joint shin_to_tarsus_left: type continuous -> fixed
- joint shin_to_tarsus_right: type continuous -> fixed
- joint toe_pitch_joint_left: type continuous -> fixed
- joint toe_pitch_joint_right: type continuous -> fixed
- joint toe_roll_joint_left: type continuous -> fixed
- joint toe_roll_joint_right: type continuous -> fixed
