Commit message: running real world experiments

File: digit/models/buff_digit/right_prosthetic.urdf (robot description, URDF)
Before this commit: robot prosthetic, 12 links, 11 joints
Links:
- link right_link2: geometry collision cylinder length=0.2 radius=0.03; visual mesh filename=meshes/link2.obj
